File: dehydration_reminder.kicad_sch (KiCad schematic)
At the start: 0 parts

Commit message: schematic completed
Parts:
- added C1: 4.7nF, Capacitor_SMD:C_0402_1005Metric, symbol Device:C
- added C11: 2.2uF, symbol Device:C
- added C3, C8: 1uF, symbol Device:C
- added C4, C5: 4.7uF, symbol Device:C
- added C6, C7: 100nF, symbol Device:C
- added C9: 0.1uF, Package_SO:SOIC-8_3.9x4.9mm_P1.27mm, symbol Device:C
- added CR1: 1N4148W-7-F, footprints2:SOD123_DIO, symbol 2026-09-20_11-48-09:1N4148W-7-F
- added D1: LED, LED_SMD:LED_0402_1005Metric_Pad0.77x0.64mm_HandSolder, symbol Device:LED
- added IC1: RT9080-33GJ5, RT9080-33GJ5:SOT94P280X100-5N, symbol RT9080-33GJ5:RT9080-33GJ5
- added J1: USB_C_Receptacle_USB2.0_16P, Connector_USB:USB_C_Receptacle_HRO_TYPE-C-31-M-12, symbol Connector:USB_C_Receptacle_USB2.0_16P
- added J2: BAT-, Connector_Wire:SolderWirePad_1x01_SMD_1x2mm, symbol Connector_Generic:Conn_01x01
- added J3: BAT+, Connector_Wire:SolderWirePad_1x01_SMD_1x2mm, symbol Connector_Generic:Conn_01x01
- added Q1: AO3400-5.8A, AO3400-5.8A:SOT95P260X140-3N, symbol AO3400-5.8A:AO3400-5.8A
- added R1, R2: 5.1K, Resistor_SMD:R_0603_1608Metric, symbol Device:R
- added R10, R9: 10K, Package_DIP:DIP-8_W7.62mm, symbol Device:R
- added R13: 100K, Package_DIP:DIP-8_W7.62mm, symbol Device:R
- added R3: 1M, Resistor_SMD:R_0603_1608Metric, symbol Device:R
- added R4: 2K, Package_DIP:DIP-8_W7.62mm, symbol Device:R
- added R5: R, Package_DIP:DIP-8_W7.62mm, symbol Device:R
- added R6: 10K, symbol Device:R
- added R7, R8: 4.7K, Package_DIP:DIP-8_W7.62mm, symbol Device:R
- added S1: JS202011SCQN, JS202011SCQN:SW_JS202011SCQN, symbol JS202011SCQN:JS202011SCQN
- added S2: PTS526_SMG15_SMTR2_LFS, PTS526_SMG15_SMTR2_LFS:SW_PTS526_SMG15_SMTR2_LFS, symbol PTS526_SMG15_SMTR2_LFS:PTS526_SMG15_SMTR2_LFS
- added U2: ESP32-C3-MINI-1U-H4, footprints3:ESP32-C3-MINI-1U_EXP, symbol 2026-09-19_12-13-52:ESP32-C3-MINI-1U-H4
- added U3: BMI270, BMI270:XDCR_BMI270, symbol BMI270:BMI270
- added U4: MCP73831-2-OT, Package_TO_SOT_SMD:SOT-23-5, symbol Battery_Management:MCP73831-2-OT
- added U5: TMB12A03, footprints4:AUDIO_TMB12A03_JHE, symbol 2026-09-19_12-16-46:TMB12A03
- added U6: USBLC6-2P6, Package_TO_SOT_SMD:SOT-666, symbol Power_Protection:USBLC6-2P6
Connections:
- new net: S2.3, S2.4, U2.21 (IO7)
- new net: C8.1, R9.2, U2.8 (EN)
- new net: C1.1, J1.SH (SHIELD), R3.1
- new net: C3.1, C5.1, IC1.1 (VIN), J3.1 (Pin_1), R13.1, U4.3 (V_{BAT})
- new net: IC1.3 (EN), S1.2
- new net: C11.1, IC1.5 (VOUT)
- new net: R5.1, U4.1 (STAT)
- new net: R4.1, U4.5 (PROG)
- new net: J1.A5 (CC1), R2.1
- new net: J1.B5 (CC2), R1.1
- new net: J1.A6 (D+), J1.B6 (D+), U6.3 (I/O2)
- new net: J1.A7 (D-), J1.B7 (D-), U6.1 (I/O1)
- new net: C9.1, R10.2, S2.1, S2.2
- new net: R13.2, S1.3
- new net: D1.1 (K), R5.2
- new net: Q1.2, R6.1
- new net: CR1.2, Q1.3, U5.2
- new net 3.3v: C6.2, C7.1, CR1.1, R10.1, R7.1, R8.1, R9.1, U2.3 (3V3), U3.12 (CSB), U3.5 (VDDIO), U3.8 (VDD), U5.1
- new net 5V: C4.1, D1.2 (A), J1.A4 (VBUS), J1.A9 (VBUS), J1.B4 (VBUS), J1.B9 (VBUS), U4.4 (V_{DD}), U6.5 (VBUS)
- new net BUZZ: Q1.1
- new net GND: C1.2, C11.2, C3.2, C4.2, C5.2, C6.1, C7.2, C8.2, C9.2, IC1.2 (GND), J1.A1 (GND), J1.A12 (GND), J1.B1 (GND), J1.B12 (GND), J2.1 (Pin_1), R1.2, R2.2, R3.2, R4.2, R6.2, S1.1, S2.G1, S2.G2, U2.1 (GND), U2.11 (GND), U2.2 (GND), U2.36 (GND), U2.37 (GND), U2.38 (GND), U2.39 (GND), U2.40 (GND), U2.41 (GND), U2.42 (GND), U2.43 (GND), U2.44 (GND), U2.45 (GND), U2.46 (GND), U2.47 (GND), U2.48 (GND), U2.49 (GND), U2.50 (GND), U2.51 (GND), U2.52 (GND), U2.53 (GND), U2.54 (GND), U2.55 (GND), U2.56 (GND), U2.57 (GND), U2.58 (GND), U2.59 (GND), U2.60 (GND), U2.61 (GND), U3.1 (SDO), U3.6 (GNDIO), U3.7 (GND), U4.2 (V_{SS}), U6.2 (GND)
- new net INT1: U2.18 (IO4), U3.4 (INT1)
- new net SCL: R7.2, U2.6 (IO3), U3.13 (SCX)
- new net SDA: R8.2, U2.5 (IO2), U3.14 (SDX)
- new net USB_DN: U2.26 (IO18), U6.6 (I/O1)
- new net USB_DP: U2.27 (IO19), U6.4 (I/O2)
- no-connect marks 0 -> 21

Commit message: final schematic made and footprints assigned
Parts:
- added C10: 0.1uF, Capacitor_SMD:C_0603_1608Metric, symbol Device:C
- added D2: RED LED, LED_SMD:LED_0402_1005Metric_Pad0.77x0.64mm_HandSolder, symbol Device:LED
- added D3: GREEN LED, LED_SMD:LED_0402_1005Metric_Pad0.77x0.64mm_HandSolder, symbol Device:LED
- added R11: 100, Resistor_SMD:R_0603_1608Metric, symbol Device:R
- added R12: 50, Resistor_SMD:R_0603_1608Metric, symbol Device:R
- added R14, R15: 100K, Resistor_SMD:R_0603_1608Metric, symbol Device:R
- C1: footprint Capacitor_SMD:C_0402_1005Metric -> Capacitor_SMD:C_0603_1608Metric
- C11, C3, C4, C5, C8: footprint (none) -> Capacitor_SMD:C_0805_2012Metric
- C6, C7: footprint (none) -> Capacitor_SMD:C_0603_1608Metric
- C9: footprint Package_SO:SOIC-8_3.9x4.9mm_P1.27mm -> Capacitor_SMD:C_0603_1608Metric
- D1: value LED -> BLUE LED
- R10, R13, R7, R8, R9: footprint Package_DIP:DIP-8_W7.62mm -> Resistor_SMD:R_0603_1608Metric
- R4: value 2K -> 4.7K; footprint Package_DIP:DIP-8_W7.62mm -> Resistor_SMD:R_0603_1608Metric
- R5: value R -> 120k; footprint Package_DIP:DIP-8_W7.62mm -> Resistor_SMD:R_0603_1608Metric
- R6: footprint (none) -> Resistor_SMD:R_0603_1608Metric
Connections:
- net 3.3v: now also C11.1, IC1.5 (VOUT)
- net 5V: now also R5.1; no longer D1.2 (A)
- net BUZZ: now also U2.13 (IO1)
- net GND: now also C10.2, D2.1 (K), D3.1 (K), R15.2
- net ADC: now reaches U2.12 (IO0)
- net ADC: now also C10.1, R14.2, R15.1
- net at U2.19 (IO5): now also R11.1
- net at U2.20 (IO6): now also R12.1
- net at C3.1, C5.1, IC1.1 (VIN)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: now also R14.1
- net at U4.1 (STAT): now also D1.1 (K); no longer R5.1
- net at R5.2: now also D1.2 (A); no longer D1.1 (K)
- new net: D3.2 (A), R12.2
- new net: D2.2 (A), R11.2
- no-connect marks 21 -> 17

Commit message: final pcb ready
Parts:
- removed C1: 4.7nF, Capacitor_SMD:C_0603_1608Metric, symbol Device:C
- removed R3: 1M, Resistor_SMD:R_0603_1608Metric, symbol Device:R
Connections:
- net GND: now also J1.SH (SHIELD)
Changed lines of the file:
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@@
-	)
-	(junction
-		(at 45.72 76.2)
-		(diameter 0)
-		(color 0 0 0 0)
 	)
 	(junction
 		(at 266.7 130.81)
-		(diameter 0)
-		(color 0 0 0 0)
-	)
-	(junction
-		(at 45.72 68.58)
 		(diameter 0)
 		(color 0 0 0 0)
@@
 	(wire
 		(pts
-			(xy 45.72 76.2) (xy 45.72 85.09)
+			(xy 45.72 66.04) (xy 45.72 77.47)
 		)
 		(stroke
@@
 	(wire
 		(pts
-			(xy 40.64 76.2) (xy 45.72 76.2)
-		)
-		(stroke
-			(width 0)
-			(type default)
-		)
-	)
-	(wire
-		(pts
 			(xy 135.89 111.76) (xy 142.24 111.76)
 		)
@@
 	(wire
 		(pts
-			(xy 45.72 68.58) (xy 50.8 68.58)
-		)
-		(stroke
-			(width 0)
-			(type default)
-		)
-	)
-	(wire
-		(pts
 			(xy 219.71 74.93) (xy 226.06 74.93)
 		)
@@
 	(wire
 		(pts
-			(xy 45.72 76.2) (xy 50.8 76.2)
-		)
-		(stroke
-			(width 0)
-			(type default)
-		)
-	)
-	(wire
-		(pts
 			(xy 266.7 87.63) (xy 266.7 90.17)
 		)
@@
 	(wire
 		(pts
-			(xy 45.72 66.04) (xy 45.72 68.58)
-		)
-		(stroke
-			(width 0)
-			(type default)
-		)
-	)
-	(wire
-		(pts
 			(xy 93.98 124.46) (xy 105.41 124.46)
 		)
@@
 		(pts
 			(xy 165.1 124.46) (xy 165.1 125.73)
-		)
-		(stroke
-			(width 0)
-			(type default)
-		)
-	)
-	(wire
-		(pts
-			(xy 40.64 68.58) (xy 45.72 68.58)
 		)
 		(stroke
@@
 	(symbol
 		(lib_id "power:GND")
-		(at 45.72 85.09 0)
+		(at 45.72 77.47 0)
 		(unit 1)
 		(body_style 1)
@@
 		(fields_autoplaced yes)
 		(property "Reference" "#PWR021"
-			(at 45.72 91.44 0)
+			(at 45.72 83.82 0)
 			(hide yes)
 			(show_name no)
@@
 		)
 		(property "Value" "GND"
-			(at 45.72 90.17 0)
+			(at 45.72 82.55 0)
 			(show_name no)
 			(do_not_autoplace no)
@@
 		)
 		(property "Footprint" ""
-			(at 45.72 85.09 0)
+			(at 45.72 77.47 0)
 			(hide yes)
 			(show_name no)
@@
 		)
 		(property "Datasheet" ""
-			(at 45.72 85.09 0)
+			(at 45.72 77.47 0)
 			(hide yes)
 			(show_name no)
@@
 		)
 		(property "Description" "Power symbol creates a global label with name \"GND\" , ground"
-			(at 45.72 85.09 0)
+			(at 45.72 77.47 0)
 			(hide yes)
 			(show_name no)
@@
 	)
 	(symbol
-		(lib_id "Device:R")
-		(at 40.64 72.39 0)
-		(unit 1)
-		(body_style 1)
-		(exclude_from_sim no)
-		(in_bom yes)
-		(on_board yes)
-		(in_pos_files yes)
-		(dnp no)
-		(property "Reference" "R3"
-			(at 36.068 71.12 0)
-			(show_name no)
-			(do_not_autoplace no)
-			(effects
-				(font
-					(size 1.27 1.27)
-				)
-				(justify left)
-			)
-		)
-		(property "Value" "1M"
-			(at 35.814 73.66 0)
-			(show_name no)
-			(do_not_autoplace no)
-			(effects
-				(font
-					(size 1.27 1.27)
-				)
-				(justify left)
-			)
-		)
-		(property "Footprint" "Resistor_SMD:R_0603_1608Metric"
-			(at 38.862 72.39 90)
-			(hide yes)
-			(show_name no)
-			(do_not_autoplace no)
-			(effects
-				(font
-					(size 1.27 1.27)
-				)
-			)
-		)
-		(property "Datasheet" ""
-			(at 40.64 72.39 0)
-			(hide yes)
-			(show_name no)
-			(do_not_autoplace no)
-			(effects
-				(font
-					(size 1.27 1.27)
-				)
-			)
-		)
-		(property "Description" "Resistor"
-			(at 40.64 72.39 0)
-			(hide yes)
-			(show_name no)
-			(do_not_autoplace no)
-			(effects
-				(font
-					(size 1.27 1.27)
-				)
-			)
-		)
-		(pin "1"
-		)
-		(pin "2"
-		)
-		(instances
-			(project "dehydration_reminder"
-				(path "/ad1c299f-56fc-4369-b208-0452ea05375d"
-					(reference "R3")
-					(unit 1)
-				)
-			)
-		)
-	)
-	(symbol
 		(lib_id "power:GND")
 		(at 138.43 101.6 180)
@@
 					(unit 1)
 				)
-			)
-		)
-	)
-	(symbol
-		(lib_id "Device:C")
-		(at 50.8 72.39 0)
-		(unit 1)
-		(body_style 1)
-		(exclude_from_sim no)
-		(in_bom yes)
-		(on_board yes)
-		(in_pos_files yes)
-		(dnp no)
-		(property "Reference" "C1"
-			(at 44.196 71.12 0)
-			(show_name no)
-			(do_not_autoplace no)
-			(effects
-				(font
-					(size 1.27 1.27)
-				)
-				(justify left)
-			)
-		)
-		(property "Value" "4.7nF"
-			(at 43.688 73.152 0)
-			(show_name no)
-			(do_not_autoplace no)
-			(effects
-				(font
-					(size 1.27 1.27)
-				)
-				(justify left)
-			)
-		)
-		(property "Footprint" "Capacitor_SMD:C_0603_1608Metric"
-			(at 51.7652 76.2 0)
-			(hide yes)
-			(show_name no)
-			(do_not_autoplace no)
-			(effects
-				(font
-					(size 1.27 1.27)
-				)
-			)
-		)
-		(property "Datasheet" ""
-			(at 50.8 72.39 0)
-			(hide yes)
-			(show_name no)
-			(do_not_autoplace no)
-			(effects
-				(font
-					(size 1.27 1.27)
-				)
-			)
-		)
-		(property "Description" "Unpolarized capacitor"
-			(at 50.8 72.39 0)
-			(hide yes)
-			(show_name no)
-			(do_not_autoplace no)
-			(effects
-				(font
-					(size 1.27 1.27)
-				)
-			)
-		)
-		(pin "1"
-		)
-		(pin "2"
-		)
-		(instances
-			(project "dehydration_reminder"
-				(path "/ad1c299f-56fc-4369-b208-0452ea05375d"
-					(reference "C1")
-					(unit 1)
-				)
